File: pcb/receiver-breakout.kicad_pcb (KiCad board)
At the start: 2 copper layers, 36 x 36 mm, 44 parts, among them P1 CONN_02X08, P2 CONN_01X02, P3 CONN_01X04, Q1 Q_NMOS_GSD, U1 74LS86, U2 74AHC2G125, U3 TLV70233DBV, U4 74LS244

Commit message: Update polystack logo to bold variant, connect i2c lines to eeprom and bump version number.
Parts:
- svg2mod (x2): footprint polystack:polystack-medium-0.4 -> polystack:polystack-bold-0.4
- moved svg2mod 0.10 mm to (164.8, 107.9) (x2)
Connections:
- PORT_IC1 pad 5: /ExpansionPort/si2c_SDA -> /ExpansionPort/i2c_SDA
- PORT_IC1 pad 6: /ExpansionPort/si2c_SCL -> /ExpansionPort/i2c_SCL
Routing:
- net /ExpansionPort/i2c_SCL: track 5.88 -> 19.8 mm
- net /ExpansionPort/i2c_SDA: track 7.56 -> 21.3 mm
- net Net-(PORT_IC1-Pad7): track 16.6 -> 18.6 mm
- net /ExpansionPort/GPIO3: track 9.52 -> 8.84 mm
Other:
- board text added: "3.3V"
- board text added: "INV"
- board text added: "ckd.tech/rcvr-bo/v3"
- board text removed: "ckd.tech/rcvr-bo/v2"

Commit message: Add license information to many files. PCB design files are CC-BY and code is MIT license.
Other:
- board text added: "Copyright 2016 Chickadee Tech LLC This work is licensed under the Creative Commons Attribution 4.0 International License. To view a copy of this license, visit http://creativecommons.org/licenses/by/4.0/ or send a letter to Creative Commons, PO Box 1866, Mountain View, CA 94042, USA."
- board text added: "Remove all Chickadee Tech LLC trademarks before making your own board. The Chickadee logo and Polystack logo are owned by Chickadee Tech LLC. You may license the Polystack logo for free by emailing support@chickadee.tech and receiving express written permission from Chickadee Tech LLC."
- board text added: "The gear logo is a mark designating open source hardware. Remove it if your design does not comply with the open source hardware definition."
Changed lines of the file:
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@@
     (links 190)
     (no_connects 0)
-    (area 129.924999 89.924999 166.075001 126.075001)
+    (area 118.127143 74.1 280.750001 191.73)
     (thickness 1.6)
-    (drawings 60)
+    (drawings 67)
     (tracks 1339)
     (zones 0)
@@
     (40 Dwgs.User user)
     (41 Cmts.User user)
-    (42 Eco1.User user hide)
-    (43 Eco2.User user hide)
+    (42 Eco1.User user)
+    (43 Eco2.User user)
     (44 Edge.Cuts user)
     (45 Margin user)
@@
       (xy 2.990233 -0.444493)) (layer B.SilkS) (width 0))
   )
+  (gr_line (start 167.43 114.75) (end 156.19 92.54) (layer Cmts.User) (width 0.2))
+  (gr_text "The gear logo is a mark designating open\nsource hardware. Remove it if your design\ndoes not comply with the open source\nhardware definition." (at 167.6 115.53) (layer Cmts.User)
+    (effects (font (size 1.5 1.5) (thickness 0.3)) (justify left))
+  )
+  (gr_line (start 163.9 107.59) (end 104.7 108.06) (layer Cmts.User) (width 0.2))
+  (gr_line (start 104.44 108.06) (end 151.4 93.39) (layer Cmts.User) (width 0.2))
+  (gr_line (start 129.87 96.75) (end 104.44 108.06) (layer Cmts.User) (width 0.2))
+  (gr_text "Remove all Chickadee Tech LLC trademarks\nbefore making your own board. The\nChickadee logo and Polystack logo\nare owned by Chickadee Tech LLC.\n\nYou may license the Polystack logo for\nfree by emailing support@chickadee.tech\nand receiving express written permission\nfrom Chickadee Tech LLC." (at 63.74 109.73) (layer Cmts.User)
+    (effects (font (size 1.5 1.5) (thickness 0.3)) (justify left))
+  )
+  (gr_text "Copyright 2016 Chickadee Tech LLC\n\nThis work is licensed under the Creative Commons Attribution 4.0 International License.\nTo view a copy of this license, visit http://creativecommons.org/licenses/by/4.0/\nor send a letter to Creative Commons, PO Box 1866, Mountain View, CA 94042, USA.\n" (at 179.1 173.95) (layer Cmts.User)
+    (effects (font (size 1.5 1.5) (thickness 0.3)) (justify left))
+  )
   (gr_text INV (at 154.7 123.87 90) (layer F.SilkS)
     (effects (font (size 1 1) (thickness 0.15)))
@@
   (gr_line (start 166 92.75) (end 166 123.25) (angle 90) (layer Edge.Cuts) (width 0.15))
   (gr_line (start 132.75 90) (end 163.25 90) (angle 90) (layer Edge.Cuts) (width 0.15))
-  (gr_text receiver-breakout (at 187.25 174.25) (layer Cmts.User)
-    (effects (font (size 5 5) (thickness 0.5)) (justify left))
+  (gr_text receiver-breakout (at 186.28 189.38) (layer Cmts.User)
+    (effects (font (size 3 3) (thickness 0.5)) (justify left))
   )
   (segment (start 153.475 106.9) (end 152.85 106.275) (width 0.1524) (layer B.Cu) (net 1))
